File: Sprayer/Board/SRX160/SRX160.kicad_pcb (KiCad board)
At the start: 2 copper layers, 172.7 x 91.4 mm, 81 parts, among them J5 12V, J6 Ground, U1 DRV8870DDA, U10 DRV8870DDA, U2 LM7805_TO220, U3 LM7809_TO220, U4 DRV8870DDA, U5 LM7805_TO220, U6 MCP6002-xP, U7 MCP6002-xP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

Commit message: update spray board
Parts:
- removed GndSensor1: WirePad, RC17Footprints:SolderWirePad16
- added D15: LED, LED_SMD:LED_0603_1608Metric, F.Cu at (127.9, 116.7)
- added D16: LED, LED_SMD:LED_0603_1608Metric, F.Cu at (114.8, 116.7)
- added D17: LED, LED_SMD:LED_0603_1608Metric, F.Cu at (176.4, 107.6)
- added D18: LED, LED_SMD:LED_0603_1608Metric, F.Cu at (167.3, 107.7)
- added D4: LED, LED_SMD:LED_0603_1608Metric, F.Cu at (154.4, 116.8)
- added D6: LED, LED_SMD:LED_0603_1608Metric, F.Cu at (140.4, 116.8)
- added FlowGnd1: WirePad, RC17Footprints:SolderWirePad16, F.Cu at (71.7, 112.4)
- added J1: 12V, RC17Footprints:PowerPin, F.Cu at (199.8, 93.2)
- added J2: Ground, RC17Footprints:PowerPin, F.Cu at (184.7, 116.7)
- added J3: Ground, RC17Footprints:PowerPin, F.Cu at (172.4, 78.3)
- added PressureGnd1: WirePad, RC17Footprints:SolderWirePad16, F.Cu at (82.8, 112.4)
- added R11: 2.2K, Resistor_SMD:R_0603_1608Metric, F.Cu at (114.7, 115.1)
- added R12: 2.2K, Resistor_SMD:R_0603_1608Metric, F.Cu at (176.4, 109.3)
- added R13: 2.2K, Resistor_SMD:R_0603_1608Metric, F.Cu at (167.3, 109.3)
- added R6: 2.2K, Resistor_SMD:R_0603_1608Metric, F.Cu at (154.3, 115.1)
- added R7: 2.2K, Resistor_SMD:R_0603_1608Metric, F.Cu at (140.4, 115.1)
- added R8: 2.2K, Resistor_SMD:R_0603_1608Metric, F.Cu at (127.8, 115.0)
- added SensorGnd1: WirePad, RC17Footprints:SolderWirePad16, F.Cu at (44.3, 99.3)
- moved J6 7.33 mm to (172.4, 90.3)
- moved J5 1.47 mm to (192.0, 88.6)
Routing:
- net M1B: track 25.8 -> 34.1 mm
- net M1A: track 23.1 -> 30.2 mm
- net S1: track 22.3 -> 26.6 mm
- net S2: track 22.2 -> 26.3 mm
- net S4: track 22.4 -> 26.5 mm
- net S3: track 22.0 -> 25.9 mm
- net Net-(D15-A): track 0.00 -> 1.74 mm
- net Net-(D17-A): track 0.00 -> 1.71 mm
- net Net-(D18-A): track 0.00 -> 1.70 mm
- net Net-(D4-A): track 0.00 -> 1.69 mm
- net Net-(D6-A): track 0.00 -> 1.69 mm
- net Net-(D16-A): track 0.00 -> 1.66 mm
- net +5V: track 172.8 -> 174.5 mm
