File: Sprayer/Board/SRX160/SRX160.kicad_pcb (KiCad board)
At the start: 2 copper layers, 172.7 x 91.4 mm, 98 parts, among them J1 12V, J2 Ground, J3 Ground, J5 12V, J6 Ground, U1 DRV8870DDA, U10 DRV8870DDA, U2 LM7805_TO220, U3 LM7809_TO220, U4 DRV8870DDA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

Commit message: pcb changes
Parts:
- added C10: 0.1uF, Capacitor_SMD:C_0603_1608Metric, F.Cu at (95.1, 62.0)
- added U11: 74HC14M, Package_SO:SOIC-14_3.9x8.7mm_P1.27mm, F.Cu at (86.3, 58.7)
- U6, U7: footprint RC17Footprints:SOIC127P600X175-8N -> Package_SO:SOIC-8_3.9x4.9mm_P1.27mm
Connections:
- A1 pad 5: FlowPin -> Net-(A1-D2)
Routing:
- net Net-(A1-D2): track 0.00 -> 40.4 mm
- net FlowPin: track 68.5 -> 32.1 mm
- net +5V: track 174.5 -> 200.6 mm
