File: Sprayer/Board/SRX160/SRX160.kicad_sch (KiCad schematic)
At the start: 33 parts, among them J5 12V, J6 Ground, U2 LM7805_TO220, U3 LM7809_TO220, U5 LM7805_TO220

Commit message: update spray board
Parts:
- added FlowGnd1, PressureGnd1: WirePad, RC17Footprints:SolderWirePad16, symbol RC17Symbols:WirePad
- added J1: 12V, RC17Footprints:PowerPin, symbol RC17Symbols:Conn_01x01
- added J2, J3: Ground, RC17Footprints:PowerPin, symbol RC17Symbols:Conn_01x01
- renumbered GndSensor1 to SensorGnd1
Connections:
- net GND: now also FlowGnd1.1, J2.1 (Pin_1), J3.1 (Pin_1), PressureGnd1.1
- net at F1.2, J5.1 (Pin_1): now also J1.1 (Pin_1)
Other:
- moved on the sheet: J6
