File: Sprayer/Board/SRX160/DRVs.kicad_sch (KiCad schematic)
At the start: 26 parts, among them U1 DRV8870DDA, U10 DRV8870DDA, U4 DRV8870DDA, U8 DRV8870DDA, U9 DRV8870DDA

Commit message: update spray board
Parts:
- added D15, D16, D17, D18, D4, D6: LED, LED_SMD:LED_0603_1608Metric, symbol RC17Symbols:LED
- added R11, R12, R13, R6, R7, R8: 2.2K, Resistor_SMD:R_0603_1608Metric, symbol RC17Symbols:R
Connections:
- net GND: now also D15.1 (K), D16.1 (K), D17.1 (K), D18.1 (K), D4.1 (K), D6.1 (K)
- net M1A: now also R13.1
- net M1B: now also R12.1
- net S1: now also R11.1
- net S2: now also R8.1
- net S3: now also R7.1
- net S4: now also R6.1
- new net: D6.2 (A), R7.2
- new net: D15.2 (A), R8.2
- new net: D4.2 (A), R6.2
- new net: D16.2 (A), R11.2
- new net: D17.2 (A), R12.2
- new net: D18.2 (A), R13.2
- no-connect marks 24 -> 26

Commit message: pcb changes
Parts:
- added C10: 0.1uF, Capacitor_SMD:C_0603_1608Metric, symbol RC17Symbols:C
- added U11: 74HC14M, Package_SO:SOIC-14_3.9x8.7mm_P1.27mm, symbol 74xx:74HC14
Connections:
- net +5V: now also C10.2, U11.14 (VCC)
- net FlowPin: now also U11.13; no longer A1.5 (D2)
- net GND: now also C10.1, U11.1, U11.11, U11.3, U11.5, U11.7 (GND), U11.9
- new net: A1.5 (D2), U11.12
- no-connect marks 26 -> 31
