File: Sprayer/Board/SRX160/Sensors.kicad_sch (KiCad schematic)
At the start: 22 parts, among them U6 MCP6002-xP, U7 MCP6002-xP

Commit message: pcb changes
Parts:
- U6, U7: footprint RC17Footprints:SOIC127P600X175-8N -> Package_SO:SOIC-8_3.9x4.9mm_P1.27mm
Changed lines of the file:
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@@
 			)
 		)
-		(property "Footprint" "RC17Footprints:SOIC127P600X175-8N"
+		(property "Footprint" "Package_SO:SOIC-8_3.9x4.9mm_P1.27mm"
 			(at 119.38 158.75 0)
 			(effects
@@
 			)
 		)
-		(property "Description" ""
+		(property "Description" "C7377"
 			(at 119.38 158.75 0)
 			(effects
@@
 			)
 		)
-		(property "Footprint" "RC17Footprints:SOIC127P600X175-8N"
+		(property "Footprint" "Package_SO:SOIC-8_3.9x4.9mm_P1.27mm"
 			(at 96.52 46.99 0)
 			(effects
@@
 			)
 		)
-		(property "Footprint" "RC17Footprints:SOIC127P600X175-8N"
+		(property "Footprint" "Package_SO:SOIC-8_3.9x4.9mm_P1.27mm"
 			(at 97.79 137.16 0)
 			(effects
@@
 			)
 		)
-		(property "Description" ""
+		(property "Description" "C7377"
 			(at 97.79 137.16 0)
 			(effects
@@
 			)
 		)
-		(property "Footprint" "RC17Footprints:SOIC127P600X175-8N"
+		(property "Footprint" "Package_SO:SOIC-8_3.9x4.9mm_P1.27mm"
 			(at 118.11 68.58 0)
 			(effects
@@
 			)
 		)
-		(property "Footprint" "RC17Footprints:SOIC127P600X175-8N"
+		(property "Footprint" "Package_SO:SOIC-8_3.9x4.9mm_P1.27mm"
 			(at 60.96 66.04 0)
 			(effects
@@
 			)
 		)
-		(property "Footprint" "RC17Footprints:SOIC127P600X175-8N"
+		(property "Footprint" "Package_SO:SOIC-8_3.9x4.9mm_P1.27mm"
 			(at 62.23 156.21 0)
 			(effects
@@
 			)
 		)
-		(property "Description" ""
+		(property "Description" "C7377"
 			(at 62.23 156.21 0)
 			(effects
